File: _autosave-dev_board_5340.sch (KiCad schematic (older format))
At the start: 73 parts, among them J1 Conn_01x04_Male, J2 USB_C_Receptacle_USB2.0, J3 Conn_01x02_Male, J4 Conn_01x23, J5 Conn_01x23, SW1 SW_Push_Dual_x2, SW2 SW_Push_Dual_x2, U1 nrf5340, U2 USBLC6-2SC6, U3 W25Q128JVS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

Commit message: test remove usb. Add base design board without trace
Parts:
- gave numbers to parts that had none: 1
Changed lines of the file:
@@
 	6000 2250 6400 2250
 $Comp
-L Device:C_Small C?
+L Device:C_Small C23
 U 1 1 60D4D75B
 P 10550 5550
-F 0 "C?" H 10642 5596 50  0000 L CNN
+F 0 "C23" H 10642 5596 50  0000 L CNN
 F 1 "5uF" H 10642 5505 50  0000 L CNN
 F 2 "Capacitor_SMD:C_0805_2012Metric" H 10550 5550 50  0001 C CNN
