File: dev_board_5340.kicad_pcb (KiCad board)
At the start: 2 copper layers, 4 parts, among them U1 nrf5340

Commit message: Refactoring. Start trace
Parts:
- added AE1: Antenna, RF_Antenna:Texas_SWRA117D_2.4GHz_Left, F.Cu at (88.9, 61.6)
- added AE2: Antenna, Connector_Coaxial:U.FL_Hirose_U.FL-R-SMT-1_Vertical, F.Cu at (84.5, 66.0)
- added C1: N.C., Capacitor_SMD:C_0805_2012Metric, F.Cu at (145.0, 53.7)
- added C10: 1uF, Capacitor_SMD:C_0402_1005Metric, F.Cu at (161.7, 78.2)
- added C11: 1uF, Capacitor_SMD:C_0402_1005Metric, F.Cu at (158.9, 78.2)
- added C12: 1uF, Capacitor_SMD:C_0402_1005Metric, F.Cu at (156.0, 78.2)
- added C13: 1uF, Capacitor_SMD:C_0402_1005Metric, F.Cu at (153.1, 78.2)
- added C14: 5uF, Capacitor_SMD:C_0805_2012Metric, F.Cu at (153.9, 75.3)
- added C15: 1uF, Capacitor_SMD:C_0805_2012Metric, F.Cu at (158.4, 71.8)
- added C16: 4.7uF, Capacitor_SMD:C_0805_2012Metric, F.Cu at (162.8, 66.8)
- added C17: 100nF, Capacitor_SMD:C_0402_1005Metric, F.Cu at (166.2, 76.2)
- added C18: 10uF, Capacitor_SMD:C_0805_2012Metric, F.Cu at (149.5, 78.3)
- added C19: C_Small, Capacitor_SMD:C_0805_2012Metric, F.Cu at (180.6, 62.1)
- added C2: 10pF, Capacitor_SMD:C_0805_2012Metric, F.Cu at (145.0, 50.7)
- added C20: C_Small, Capacitor_SMD:C_0805_2012Metric, F.Cu at (171.7, 65.1)
- added C21: 100pF, Capacitor_SMD:C_0805_2012Metric, F.Cu at (171.7, 68.2)
- added C22: 100pF, Capacitor_SMD:C_0805_2012Metric, F.Cu at (176.2, 68.2)
- added C23: 100pF, Capacitor_SMD:C_0805_2012Metric, F.Cu at (162.8, 71.2)
- added C24: 100pF, Capacitor_SMD:C_0805_2012Metric, F.Cu at (145.0, 75.3)
- added C25: 10uF, Capacitor_SMD:C_1206_3216Metric, F.Cu at (162.9, 56.0)
- added C26: 10uF, Capacitor_SMD:C_1206_3216Metric, F.Cu at (168.5, 53.7)
- added C27: 1uF, Capacitor_SMD:C_0805_2012Metric, F.Cu at (149.5, 81.3)
- added C28: 1uF, Capacitor_SMD:C_0402_1005Metric, F.Cu at (160.4, 76.2)
- added C29: 2.2nF, Capacitor_SMD:C_0402_1005Metric, F.Cu at (157.6, 76.2)
- added C3: 10pF, Capacitor_SMD:C_0805_2012Metric, F.Cu at (145.0, 81.3)
- added C4: C_Small, Capacitor_SMD:C_0805_2012Metric, F.Cu at (149.5, 75.3)
- added C5: 1uF, Capacitor_SMD:C_0402_1005Metric, F.Cu at (167.8, 74.2)
- added C6: 1uF, Capacitor_SMD:C_0402_1005Metric, F.Cu at (153.1, 80.1)
- added C7: 1uF, Capacitor_SMD:C_0805_2012Metric, F.Cu at (145.0, 78.3)
- added C8: 1uF, Capacitor_SMD:C_0402_1005Metric, F.Cu at (163.3, 76.2)
- added C9: 1uF, Capacitor_SMD:C_0402_1005Metric, F.Cu at (164.6, 78.2)
- added D4: LED, Diode_SMD:D_0805_2012Metric, F.Cu at (176.2, 59.1)
- added D5: LED, Diode_SMD:D_0805_2012Metric, F.Cu at (171.7, 60.2)
- added D6: LED, Diode_SMD:D_0805_2012Metric, F.Cu at (167.3, 66.8)
- added D7: LED, Diode_SMD:D_0805_2012Metric, F.Cu at (176.2, 65.1)
- added F1: Fuse, Fuse:Fuse_1206_3216Metric, F.Cu at (162.8, 63.6)
- added J1: Conn_01x04_Male, Connector_PinHeader_2.54mm:PinHeader_1x04_P2.54mm_Vertical, F.Cu at (161.8, 44.4)
- added J2: USB_C_Receptacle_USB2.0, Connector_USB:USB_C_Receptacle_XKB_U262-16XN-4BVC11, F.Cu at (81.3, 110.5)
- added J3: Conn_01x02_Male, Connector_PinHeader_2.54mm:PinHeader_1x02_P2.54mm_Vertical, F.Cu at (117.0, 45.8)
- added J4: Conn_01x23, Connector_PinHeader_2.54mm:PinHeader_1x23_P2.54mm_Vertical, F.Cu at (73.7, 57.1)
- added J5: Conn_01x23, Connector_PinHeader_2.54mm:PinHeader_1x23_P2.54mm_Vertical, F.Cu at (104.1, 57.1)
- added L1: 2.2nH, Inductor_SMD:L_1206_3216Metric, F.Cu at (157.2, 64.1)
- added L2: 10uH, Inductor_SMD:L_1206_3216Metric, F.Cu at (151.4, 67.4)
- added L3: 10uH, Inductor_SMD:L_1206_3216Metric, F.Cu at (145.7, 67.4)
- added R1: 3k5, Resistor_SMD:R_0402_1005Metric, F.Cu at (157.0, 54.1)
- added R10: 0R0, Resistor_SMD:R_0402_1005Metric, F.Cu at (157.7, 56.1)
- added R11: 0R0, Resistor_SMD:R_0402_1005Metric, F.Cu at (165.0, 74.2)
- added R12: 2R2, Resistor_SMD:R_1206_3216Metric, F.Cu at (159.1, 60.3)
- added R13: 2k, Resistor_SMD:R_0402_1005Metric, F.Cu at (162.0, 74.2)
- added R14: 10R, Resistor_SMD:R_1206_3216Metric, F.Cu at (164.7, 60.3)
- added R15: 10R, Resistor_SMD:R_1206_3216Metric, F.Cu at (168.5, 57.0)
- added R16: 1k5, Resistor_SMD:R_0402_1005Metric, F.Cu at (169.4, 72.2)
- added R17: 3k5, Resistor_SMD:R_0402_1005Metric, F.Cu at (148.7, 50.1)
- added R18: 3k5, Resistor_SMD:R_0402_1005Metric, F.Cu at (166.5, 72.2)
- added R19: 3k5, Resistor_SMD:R_0402_1005Metric, F.Cu at (152.4, 63.4)
- added R2: 3k5, Resistor_SMD:R_0402_1005Metric, F.Cu at (157.0, 52.1)
- added R3: 3k.5, Resistor_SMD:R_0402_1005Metric, F.Cu at (148.7, 54.1)
- added R4: R_Small, Resistor_SMD:R_0805_2012Metric, F.Cu at (167.2, 69.8)
- added R5: R_Small, Resistor_SMD:R_0805_2012Metric, F.Cu at (173.5, 53.5)
- added R6: R_Small, Resistor_SMD:R_0402_1005Metric, F.Cu at (148.7, 52.1)
- added R7: 3k, Resistor_SMD:R_0402_1005Metric, F.Cu at (147.2, 56.2)
- added R8: 3k5, Resistor_SMD:R_0402_1005Metric, F.Cu at (144.2, 56.2)
- added R9: 2k0, Resistor_SMD:R_0402_1005Metric, F.Cu at (157.0, 50.1)
- added SW1: SW_Push_Dual_x2, Button_Switch_SMD:SW_Push_1P1T_NO_CK_KSC6xxJ, F.Cu at (98.4, 108.6)
- added SW2: SW_Push_Dual_x2, Button_Switch_SMD:SW_Push_1P1T_NO_CK_KSC6xxJ, F.Cu at (90.8, 108.6)
- added U2: USBLC6-2SC6, Package_TO_SOT_SMD:SOT-23-6, F.Cu at (81.9, 102.2)
- added U3: W25Q128JVS, Package_SO:SOIC-8_5.23x5.23mm_P1.27mm, F.Cu at (95.9, 83.2)
- added U4: AZ1117-3.3, Package_TO_SOT_SMD:SOT-223, F.Cu at (97.2, 59.3)
- added Y1: Crystal_GND24_Small, Crystal:Crystal_SMD_3225-4Pin_3.2x2.5mm, F.Cu at (81.9, 76.2)
- added Y2: Crystal_Small, Crystal:Crystal_SMD_3215-2Pin_3.2x1.5mm, F.Cu at (145.3, 72.0)
- D1: value SFH4356P -> ASMT-YTC2-0AA02; footprint LED_THT:LED_D3.0mm_IRBlack -> LED_SMD:LED_Avago_PLCC6_3x2.8mm
- D2, D3: value SFH4356P -> LED; footprint LED_THT:LED_D3.0mm_IRBlack -> Diode_SMD:D_0805_2012Metric
- moved D2 53.4 mm to (176.2, 62.1)
- moved D3 51.2 mm to (180.6, 59.1)
- moved D1 36.0 mm to (91.6, 70.9)
- moved U1 34.0 mm to (87.6, 81.9), turned to 90 degrees
Connections:
- D1 pad 1: Net-(D1-Pad1) -> GNDREF
- D1 pad 2: Net-(D1-Pad2) -> GNDREF
- D2 pad 1: Net-(D2-Pad1) -> GNDREF
- D3 pad 1: Net-(D3-Pad1) -> GNDREF
- U1 pad A17: Net-(U1-PadA17) -> /P1.13
- U1 pad A19: Net-(U1-PadA19) -> VDD
- U1 pad A25: Net-(U1-PadA25) -> GNDREF
- U1 pad AB2: Net-(U1-PadAB2) -> /P0.6
- U1 pad AC1: Net-(U1-PadAC1) -> VDD
- U1 pad AC31: Net-(U1-PadAC31) -> (no net)
- U1 pad AD2: Net-(U1-PadAD2) -> /P0.7
- U1 pad AE1: Net-(U1-PadAE1) -> /P1.2
- U1 pad AE31: Net-(U1-PadAE31) -> /P0.28
- U1 pad AF2: Net-(U1-PadAF2) -> /P1.3
- U1 pad AG1: Net-(U1-PadAG1) -> VDD
- U1 pad AG31: Net-(U1-PadAG31) -> (no net)
- U1 pad AH2: Net-(U1-PadAH2) -> /P0.8
- U1 pad AJ1: Net-(U1-PadAJ1) -> /P0.9
- U1 pad AJ31: Net-(U1-PadAJ31) -> VDD
- U1 pad AK10: Net-(U1-PadAK10) -> /QSPI_2
- U1 pad AK12: Net-(U1-PadAK12) -> /QSPI_CLK
- U1 pad AK14: Net-(U1-PadAK14) -> /QSPI_CS
- U1 pad AK16: (no net) -> /R_LED
- U1 pad AK18: Net-(U1-PadAK18) -> /B_LED
- U1 pad AK2: Net-(U1-PadAK2) -> /P0.10
- U1 pad AK20: Net-(U1-PadAK20) -> /P0.23
- U1 pad AK22: Net-(U1-PadAK22) -> /P1.5
- U1 pad AK24: Net-(U1-PadAK24) -> /P1.7
- U1 pad AK26: Net-(U1-PadAK26) -> /P1.9
- U1 pad AK28: Net-(U1-PadAK28) -> /P0.25
- U1 pad AK30: Net-(U1-PadAK30) -> /P0.27
- U1 pad AK4: Net-(U1-PadAK4) -> /P0.11
- U1 pad AK6: Net-(U1-PadAK6) -> /P0.12
- U1 pad AK8: Net-(U1-PadAK8) -> /QSPI_1
- U1 pad AL11: Net-(U1-PadAL11) -> VDD
- U1 pad AL13: Net-(U1-PadAL13) -> (no net)
- U1 pad AL15: Net-(U1-PadAL15) -> /G_LED
- U1 pad AL17: Net-(U1-PadAL17) -> VDD
- U1 pad AL19: Net-(U1-PadAL19) -> /P1.4
- U1 pad AL21: Net-(U1-PadAL21) -> /P1.6
- U1 pad AL23: Net-(U1-PadAL23) -> VDD
- U1 pad AL25: Net-(U1-PadAL25) -> VDD
- U1 pad AL27: Net-(U1-PadAL27) -> /P0.24
- U1 pad AL29: Net-(U1-PadAL29) -> /P0.26
- U1 pad AL3: Net-(U1-PadAL3) -> VDD
- U1 pad AL5: Net-(U1-PadAL5) -> /QSPI_0
- U1 pad AL7: Net-(U1-PadAL7) -> VDD
- U1 pad AL9: Net-(U1-PadAL9) -> /QSPI_3
- U1 pad B12: Net-(U1-PadB12) -> GNDREF
- U1 pad B14: Net-(U1-PadB14) -> /P1.15
- U1 pad B16: Net-(U1-PadB16) -> /P1.14
- U1 pad B18: Net-(U1-PadB18) -> /P1.12
- U1 pad B2: Net-(U1-PadB2) -> (no net)
- U1 pad B20: Net-(U1-PadB20) -> /P1.11
- U1 pad B22: Net-(U1-PadB22) -> /P0.31
- U1 pad B24: Net-(U1-PadB24) -> /P0.30
- U1 pad B26: Net-(U1-PadB26) -> GNDREF
- U1 pad B28: Net-(U1-PadB28) -> VDD
- U1 pad B4: Net-(U1-PadB4) -> (no net)
- U1 pad B8: Net-(U1-PadB8) -> VDD
- U1 pad C1: Net-(U1-PadC1) -> VDD
- U1 pad E1: Net-(U1-PadE1) -> VDD
- U1 pad E31: (no net) -> VDD
- U1 pad G1: Net-(U1-PadG1) -> GNDREF
- U1 pad G31: Net-(U1-PadG31) -> Net-(U1-PadA27)
- U1 pad H2: Net-(U1-PadH2) -> GNDREF
- U1 pad J1: Net-(U1-PadJ1) -> (no net)
- U1 pad J31: Net-(U1-PadJ31) -> GNDREF
- U1 pad L1: Net-(U1-PadL1) -> VDD
- U1 pad M2: Net-(U1-PadM2) -> /P1.0
- U1 pad N31: Net-(U1-PadN31) -> VDD
- U1 pad P2: Net-(U1-PadP2) -> /P1.1
- U1 pad R31: Net-(U1-PadR31) -> /P1.10
- U1 pad U1: Net-(U1-PadU1) -> VDD
- U1 pad U31: Net-(U1-PadU31) -> /P0.29
- U1 pad V2: Net-(U1-PadV2) -> /P0.4
- U1 pad VSS: (no net) -> GNDREF
- U1 pad Y2: Net-(U1-PadY2) -> /P0.5

Commit message: test remove usb. Add base design board without trace
Parts:
- removed C24: 100pF, Capacitor_SMD:C_0805_2012Metric
- C10, C11, C12, C13, C5, C6, C7, C8, C9: moved to B.Cu
- C21, C22: value 100pF -> 200pF
- C23: value 100pF -> 5uF
- D2, D3, D4, D5, D6, D7: footprint Diode_SMD:D_0805_2012Metric -> Diode_SMD:D_0603_1608Metric
- R1, R17, R18, R19, R2, R3, R6, R7, R8: footprint Resistor_SMD:R_0402_1005Metric -> Resistor_SMD:R_0603_1608Metric
- moved D3 106.3 mm to (80.0, 93.3)
- moved D2 100.5 mm to (83.8, 101.6), turned to 180 degrees
- moved C19 100.0 mm to (86.4, 95.6), turned to 90 degrees
- moved R15 99.1 mm to (76.8, 94.6), turned to 270 degrees
- moved R5 97.0 mm to (89.5, 102.0), turned to 270 degrees
- moved F1 93.5 mm to (76.8, 100.2), turned to 270 degrees
- moved R14 88.6 mm to (83.2, 95.1), turned to 270 degrees
- moved C20 88.2 mm to (88.9, 95.6), turned to 90 degrees
- moved R16 87.3 mm to (84.3, 91.8), turned to 180 degrees
- moved R4 86.4 mm to (87.0, 101.9), turned to 270 degrees
- moved C17 84.2 mm to (82.1, 80.6), turned to 90 degrees
- moved C5 84.1 mm to (84.5, 85.1)
- moved R12 83.9 mm to (80.5, 89.5)
- moved C28 83.8 mm to (76.8, 81.3)
- moved C22 83.7 mm to (96.5, 94.0), turned to 270 degrees
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Connections:
- C23 pad 1: GNDREF -> Net-(C23-Pad1)
- C23 pad 2: Net-(C21-Pad2) -> GNDREF
- J4 pad 13: (no net) -> /P1.8
- R13 pad 2: Net-(R13-Pad2) -> Net-(C23-Pad1)
- SW2 pad 1: Net-(R13-Pad2) -> Net-(C23-Pad1)
- U1 pad AL23: VDD -> /P1.8
Other:
- net class QFN added: clearance 0.1, trace_width 0.2, via_dia 0.8, via_drill 0.4
- rule trace_min: 0.2 -> 0.1
- rule via_min_size: 0.4 -> 0.2
